File: Hardware/Basisboard Klemme/Basisboard_Klemme.brd (EAGLE design)
At the start: 85 x 65 mm, 37 parts, among them IC1 MEGA8-AI, IC2 MCP2551SO8, Q1 16M, Q2 16M, U1 TSR_1-24_, X1 MEBP 8-8G, X2 MEBP 8-8G

Commit message: REV0101
Parts:
- R4, R5: value 680 -> 1k
- X5: device con-lstb:MA03-2 -> con-harting-ml:ML6
- moved U$2 16.0 mm to (55.9, 55.0)
- moved C4 7.01 mm to (56.5, 40.7)
- moved IC1 5.14 mm to (41.7, 34.9)
- moved X5 4.87 mm to (54.1, 28.8)
- moved R1 3.70 mm to (39.1, 42.6)
- moved Q1 3.22 mm to (29.0, 36.1)
- moved C1 3.18 mm to (32.7, 38.5)
- moved C2 3.18 mm to (32.7, 33.4)
- moved C5 2.20 mm to (52.6, 17.3)
- moved C6 2.20 mm to (52.6, 12.2)
- moved Q2 2.19 mm to (56.3, 14.7)
- moved C3 0.32 mm to (31.6, 27.0)
Routing:
- net VCC: track 183.1 -> 196.7 mm
- net STATUS: track 55.9 -> 63.0 mm
- net MOSI: track 23.0 -> 29.3 mm
- net SCL: track 33.9 -> 28.0 mm
- net SDA: track 32.1 -> 26.3 mm
- net 17/A3: track 30.4 -> 24.5 mm
- net 16/A2: track 28.6 -> 22.9 mm
- net SCK: track 18.7 -> 24.0 mm
- net MISO: track 15.7 -> 21.0 mm
- net 15/A1: track 32.7 -> 28.0 mm
- net 14/A0: track 32.0 -> 27.4 mm
- net 5: track 28.8 -> 24.4 mm
- net CS: track 9.18 -> 12.9 mm
- net 6: track 27.4 -> 23.7 mm
- net INT: track 23.6 -> 26.9 mm
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Other:
- board text added: "CAN Basisboard 2020 - Version 1.1"
- board text removed: "CAN Basisboard 2020 - Version 1.0"
