File: Hardware/Basisboard Klemme/Basisboard_Klemme.sch (EAGLE design)
At the start: 35 parts, among them IC1 MEGA8-AI, IC2 MCP2551SO8, Q1 16M, Q2 16M, U1 TSR_1-24_, X1 MEBP 8-8G, X2 MEBP 8-8G

Commit message: REV0101
Parts:
- C1, C2, C5, C6: LCSC_PART (none) -> C313096
- C3, C4: LCSC_PART (none) -> C24497
- IC1: LCSC_PART (none) -> C132230
- IC2: LCSC_PART (none) -> C49558
- IC3: LCSC_PART (none) -> C153782
- POWER: LCSC_PART (none) -> C88326
- R1, R2: LCSC_PART (none) -> C17902
- R3: LCSC_PART (none) -> C17909
- R4, R5: value 680 -> 1k; LCSC_PART (none) -> C4410
- STATUS: LCSC_PART (none) -> C84273
- X5: device con-lstb:MA03-2 -> con-harting-ml:ML6
